File: DIY/STM32 Board/untitled.brd (EAGLE design)
At the start: 100 x 80 mm, 13 parts, among them IC1 MCP1703DB, Q1 16 MHz, U1 STM32103RBT6

Commit message: DIY ++
Parts:
- removed IC1: MCP1703DB, linear:SOT223
- added C10, C11: 10 uF, rcl:A/3216-18W
- added C8, C9: 100 nF, resistor:C1206
- added IC2: REG1117, burr-brown:SOT223
- moved C3 87.9 mm to (45.5, 45.0)
- moved Q1 79.1 mm to (57.5, 39.0), turned to 270 degrees
- moved C1 66.8 mm to (30.5, 45.0)
- moved C4 17.6 mm to (-33.0, 17.8)
- moved C5 17.6 mm to (-40.6, 17.8)
- moved U1 16.5 mm to (38.0, 39.0), turned to 90 degrees
- moved R1 13.0 mm to (-38.1, 34.3)
- moved JP2 6.42 mm to (2.50, 37.1)
- moved C2 2.54 mm to (-31.8, 24.1)
- moved C6 2.54 mm to (-38.1, 24.1)
- moved C7 2.54 mm to (-44.5, 24.1)
- moved JP1 2.54 mm to (-17.8, 35.6)
Connections:
- net +3V3: now also C1.2, C11.+, C9.1, IC2.2; no longer C1.1
- net +5V: now also C10.+, C8.2, IC2.3
- net GND: now also C1.1, C10.-, C11.-, C6.2, C7.2, C8.1, C9.2, IC2.1; no longer C1.2, C6.1, C7.1
- net N$1: now also C6.1; no longer C6.2
- net N$2: now also C7.1; no longer C7.2
Routing:
- net LCD_DB5: track 41.6 -> 43.4 mm
- net LCD_DB6: track 42.1 -> 43.7 mm
- net LCD_DB4: track 41.7 -> 43.0 mm
- net LCD_DB7: track 43.0 -> 44.0 mm
- net LCD_DB3: track 41.9 -> 42.6 mm
- added copper zone on layer 1, net GND
Other:
- board size 100 x 80 mm -> 100 x 78 mm

Commit message: ++
Parts:
- C1, C8: value 100 nF -> 10 uF; device resistor:C1206 -> rcl:A/3216-18W
- C10, C11: value 10 uF -> 30 pF; device rcl:A/3216-18W -> resistor:C1206
- C2: value 10 μF -> 100 nF
- C6, C7: value 30 pF -> 100 nF
- C9: value 100 nF -> 10 μF
- moved C3 90.3 mm to (-40.6, 17.8)
- moved C5 90.3 mm to (45.5, 45.0)
- moved C6 84.1 mm to (45.5, 33.0)
- moved C7 77.8 mm to (30.5, 45.0)
- moved C9 77.8 mm to (-31.8, 24.1)
- moved C2 62.9 mm to (30.5, 33.0)
- moved C8 62.4 mm to (-31.8, 36.8)
- moved C1 56.5 mm to (-25.4, 36.8)
- moved C10 18.0 mm to (-38.1, 24.1)
- moved C11 18.0 mm to (-44.5, 24.1)
- renumbered IC2 to IC1
Connections:
- net +3V3: now also C6.1, C7.2, C8.+; no longer C1.2, C11.+, C2.1
- net +5V: now also C1.+, C2.2; no longer C10.+, C8.2
- net GND: now also C1.-, C10.2, C11.2, C2.1, C7.1, C8.-; no longer C1.1, C10.-, C11.-, C2.2, C7.2, C8.1
- net N$1: now also C10.1; no longer C6.1
- net N$2: now also C11.1; no longer C7.1
Changed lines of the file:
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@@
 </autorouter>
 <elements>
-<element name="C1" library="resistor" package="C1206" value="100 nF" x="30.5" y="45"/>
-<element name="C10" library="rcl" package="A/3216-18W" value="10 uF" x="-25.4" y="36.83"/>
-<element name="C11" library="rcl" package="A/3216-18W" value="10 uF" x="-31.75" y="36.83"/>
-<element name="C2" library="resistor" package="C1206" value="10 μF" x="-31.75" y="24.13"/>
-<element name="C3" library="resistor" package="C1206" value="100 nF" x="45.5" y="45"/>
+<element name="C7" library="resistor" package="C1206" value="100 nF" x="30.5" y="45"/>
+<element name="C1" library="rcl" package="A/3216-18W" value="10 uF" x="-25.4" y="36.83"/>
+<element name="C8" library="rcl" package="A/3216-18W" value="10 uF" x="-31.75" y="36.83"/>
+<element name="C9" library="resistor" package="C1206" value="10 μF" x="-31.75" y="24.13"/>
+<element name="C5" library="resistor" package="C1206" value="100 nF" x="45.5" y="45"/>
 <element name="C4" library="resistor" package="C1206" value="100 nF" x="-33.02" y="17.78"/>
-<element name="C5" library="resistor" package="C1206" value="100 nF" x="-40.64" y="17.78"/>
-<element name="C6" library="resistor" package="C1206" value="30 pF" x="-38.1" y="24.13"/>
-<element name="C7" library="resistor" package="C1206" value="30 pF" x="-44.45" y="24.13"/>
-<element name="C8" library="resistor" package="C1206" value="100 nF" x="30.52" y="33.03"/>
-<element name="C9" library="resistor" package="C1206" value="100 nF" x="45.5" y="33"/>
-<element name="IC2" library="burr-brown" package="SOT223" value="REG1117" x="-33.02" y="6.35">
+<element name="C3" library="resistor" package="C1206" value="100 nF" x="-40.64" y="17.78"/>
+<element name="C10" library="resistor" package="C1206" value="30 pF" x="-38.1" y="24.13"/>
+<element name="C11" library="resistor" package="C1206" value="30 pF" x="-44.45" y="24.13"/>
+<element name="C2" library="resistor" package="C1206" value="100 nF" x="30.52" y="33.03"/>
+<element name="C6" library="resistor" package="C1206" value="100 nF" x="45.5" y="33"/>
+<element name="IC1" library="burr-brown" package="SOT223" value="REG1117" x="-33.02" y="6.35">
 <attribute name="MPN" value="REG1117" x="-33.02" y="6.35" size="1.778" layer="27" display="off"/>
 <attribute name="OC_FARNELL" value="1097566" x="-33.02" y="6.35" size="1.778" layer="27" display="off"/>
@@
 <contactref element="U1" pad="63"/>
 <contactref element="U1" pad="18"/>
-<contactref element="C6" pad="2"/>
-<contactref element="C7" pad="2"/>
+<contactref element="C10" pad="2"/>
+<contactref element="C11" pad="2"/>
 <contactref element="JP1" pad="3"/>
 <contactref element="JP2" pad="1"/>
 <contactref element="JP2" pad="2"/>
 <contactref element="JP2" pad="19"/>
-<contactref element="C2" pad="2"/>
-<contactref element="C1" pad="1"/>
+<contactref element="C9" pad="2"/>
+<contactref element="C7" pad="1"/>
+<contactref element="C5" pad="2"/>
+<contactref element="C4" pad="2"/>
 <contactref element="C3" pad="2"/>
-<contactref element="C4" pad="2"/>
-<contactref element="C5" pad="2"/>
-<contactref element="IC2" pad="1"/>
-<contactref element="C8" pad="1"/>
-<contactref element="C9" pad="2"/>
-<contactref element="C10" pad="-"/>
-<contactref element="C11" pad="-"/>
+<contactref element="IC1" pad="1"/>
+<contactref element="C2" pad="1"/>
+<contactref element="C6" pad="2"/>
+<contactref element="C1" pad="-"/>
+<contactref element="C8" pad="-"/>
 <polygon width="0.3" layer="1">
 <vertex x="-0.5" y="78.5"/>
@@
 <contactref element="JP2" pad="4"/>
 <contactref element="JP2" pad="3"/>
-<contactref element="IC2" pad="3"/>
-<contactref element="C8" pad="2"/>
-<contactref element="C10" pad="+"/>
+<contactref element="IC1" pad="3"/>
+<contactref element="C2" pad="2"/>
+<contactref element="C1" pad="+"/>
 <wire x1="2.5" y1="12.97" x2="31.92" y2="33.03" width="0" layer="19" extent="1-1"/>
 <wire x1="-30.7086" y1="3.2004" x2="2.5" y2="12.97" width="0" layer="19" extent="1-1"/>
@@
 </signal>
 <signal name="+3V3">
-<contactref element="C2" pad="1"/>
-<contactref element="C1" pad="2"/>
+<contactref element="C9" pad="1"/>
+<contactref element="C7" pad="2"/>
 <contactref element="U1" pad="13"/>
 <contactref element="U1" pad="1"/>
@@
 <contactref element="U1" pad="48"/>
 <contactref element="U1" pad="32"/>
+<contactref element="C5" pad="1"/>
+<contactref element="C4" pad="1"/>
 <contactref element="C3" pad="1"/>
-<contactref element="C4" pad="1"/>
-<contactref element="C5" pad="1"/>
-<contactref element="IC2" pad="2"/>
-<contactref element="C9" pad="1"/>
-<contactref element="C11" pad="+"/>
+<contactref element="IC1" pad="2"/>
+<contactref element="C6" pad="1"/>
+<contactref element="C8" pad="+"/>
 <wire x1="40.75" y1="44.75" x2="44.1" y2="45" width="0" layer="19" extent="1-1"/>
 <wire x1="43.75" y1="41.25" x2="44.1" y2="45" width="0" layer="19" extent="1-1"/>
@@
 <contactref element="U1" pad="5"/>
 <contactref element="Q1" pad="1"/>
-<contactref element="C6" pad="1"/>
+<contactref element="C10" pad="1"/>
 <wire x1="43.75" y1="37.25" x2="57.5" y2="41.413" width="0" layer="19" extent="1-1"/>
 <wire x1="-39.5" y1="24.13" x2="43.75" y2="37.25" width="0" layer="19" extent="1-1"/>
@@
 <contactref element="Q1" pad="2"/>
 <contactref element="R1" pad="1"/>
-<contactref element="C7" pad="1"/>
+<contactref element="C11" pad="1"/>
 <wire x1="-39.522" y1="34.29" x2="57.5" y2="36.587" width="0" layer="19" extent="1-1"/>
 <wire x1="-45.85" y1="24.13" x2="-39.522" y2="34.29" width="0" layer="19" extent="1-1"/>
